File: pcb/3x10t6m.kicad_pcb (KiCad board)
At the start: 2 copper layers, 276.5 x 107.2 mm, 89 parts, among them J1 Conn_01x03, J2 Conn_01x05, SW1 SW_PUSH, SW10 SW_PUSH, SW11 SW_PUSH, SW12 SW_PUSH, SW13 SW_PUSH, SW14 SW_PUSH, SW15 SW_PUSH, SW16 SW_PUSH, SW17 SW_PUSH, SW18 SW_PUSH, SW19 SW_PUSH, SW2 SW_PUSH, SW20 SW_PUSH, SW21 SW_PUSH, SW22 SW_PUSH, SW23 SW_PUSH, SW24 SW_PUSH, SW25 SW_PUSH, SW26 SW_PUSH, SW27 SW_PUSH, SW28 SW_PUSH, SW29 SW_PUSH, SW3 SW_PUSH, SW30 SW_PUSH, SW31 SW_PUSH, SW32 SW_PUSH, SW33 SW_PUSH, SW34 SW_PUSH, SW35 SW_PUSH, SW36 SW_PUSH, SW37 SW_PUSH, SW38 SW_PUSH, SW39 SW_PUSH, SW4 SW_PUSH, SW40 SW_PUSH, SW41 SW_PUSH, SW42 SW_PUSH, SW43 SW_PUSH, SW44 SW_SPDT, SW5 SW_PUSH, SW6 SW_PUSH, SW7 SW_PUSH, SW8 SW_PUSH, SW9 SW_PUSH

Commit message: add firmware stuff
Parts:
- removed J1: Conn_01x03, Connector_JST:JST_PH_S3B-PH-SM4-TB_1x03-1MP_P2.00mm_Horizontal
- removed J2: Conn_01x05, Connector_PinHeader_2.54mm:PinHeader_1x05_P2.54mm_Vertical
- removed SW44: SW_SPDT, footprints:CUS-12TB
- A1: value ProMicro -> promicro
- moved D1 3.14 mm to (36.3, 72.0)
- moved SW43 1.29 mm to (147.8, 116.7)
Connections:
- A1 pad 1: CS -> LED
- A1 pad 13: unconnected-(A1-Pad13) -> Net-(A1-Pad13)
- A1 pad 2: unconnected-(A1-Pad2) -> Net-(A1-Pad2)
- A1 pad 5: mosi -> Net-(A1-Pad5)
- A1 pad 6: sck -> Net-(A1-Pad6)
Routing:
- net GND: track 190.3 -> 60.8 mm, vias 6 -> 1
- net Net-(J1-Pad2): track 113.6 -> 0.00 mm, vias 6 -> 0
- net VCC: track 63.1 -> 0.00 mm, vias 1 -> 0
- net mosi: track 51.1 -> 0.00 mm, vias 1 -> 0
- net CS: track 47.1 -> 0.00 mm, vias 1 -> 0
- net sck: track 43.9 -> 0.00 mm, vias 1 -> 0
- net Net-(A1-Pad24): track 10.4 -> 0.00 mm, vias 1 -> 0
- net col4: track 324.3 -> 320.4 mm, vias 8 -> 6
- net row0: track 118.0 -> 115.0 mm
- net col3: track 304.1 -> 301.9 mm, vias 4 -> 3
- net col5: track 311.5 -> 313.6 mm, vias 6 -> 5
- net row6: track 185.1 -> 183.7 mm
- net reset: track 36.6 -> 37.9 mm
Other:
- outline, holes or cut-outs redrawn
